File: _autosave-ai03-pcb-guide.sch (KiCad schematic (older format))
At the start: 9 parts

Commit message: Update _autosave-ai03-pcb-guide.sch
Parts:
- added C? (x2): 22pF, symbol Device:C_Small
- added R?: 10k, symbol Device:R_Small
- added SW?: SW_Push, symbol Switch:SW_Push
- added Y?: 16MHz, symbol Device:Crystal_GND24_Small
- C?: value C_Small -> 1uF
- C?: value C_Small -> 10uF
- C? (x3): value C_Small -> 0.1uF
- R? (x2): value R_Small -> 22
Connections:
- net labels added: D+, D-
- wire segments 15 -> 46
Changed lines of the file:
@@
 P 3400 2950
 F 0 "R?" V 3204 2950 50  0000 C CNN
-F 1 "R_Small" V 3295 2950 50  0000 C CNN
+F 1 "22" V 3295 2950 50  0000 C CNN
 F 2 "" H 3400 2950 50  0001 C CNN
 F 3 "~" H 3400 2950 50  0001 C CNN
@@
 P 3000 3050
 F 0 "R?" V 2804 3050 50  0000 C CNN
-F 1 "R_Small" V 2895 3050 50  0000 C CNN
+F 1 "22" V 2895 3050 50  0000 C CNN
 F 2 "" H 3000 3050 50  0001 C CNN
 F 3 "~" H 3000 3050 50  0001 C CNN
@@
 P 3350 3350
 F 0 "C?" H 3442 3396 50  0000 L CNN
-F 1 "C_Small" H 3442 3305 50  0000 L CNN
+F 1 "1uF" H 3442 3305 50  0000 L CNN
 F 2 "" H 3350 3350 50  0001 C CNN
 F 3 "~" H 3350 3350 50  0001 C CNN
@@
 $Comp
 L Device:C_Small C?
+U 1 1 66998AAD
+P 2750 4250
+F 0 "C?" H 2842 4296 50  0000 L CNN
+F 1 "0.1uF" H 2842 4205 50  0000 L CNN
+F 2 "" H 2750 4250 50  0001 C CNN
+F 3 "~" H 2750 4250 50  0001 C CNN
+	1    2750 4250
+	1    0    0    -1
+$EndComp
+$Comp
+L Device:C_Small C?
+U 1 1 669A1692
+P 2250 4250
+F 0 "C?" H 2342 4296 50  0000 L CNN
+F 1 "0.1uF" H 2342 4205 50  0000 L CNN
+F 2 "" H 2250 4250 50  0001 C CNN
+F 3 "~" H 2250 4250 50  0001 C CNN
+	1    2250 4250
+	1    0    0    -1
+$EndComp
+Wire Wire Line
+	2500 4150 2250 4150
+Connection ~ 2250 4150
+Wire Wire Line
+	2500 4350 2500 4450
+Connection ~ 2250 4350
+Wire Wire Line
+	2250 4350 2500 4350
+Connection ~ 2500 4150
+Connection ~ 2750 4150
+Connection ~ 2500 4350
+Connection ~ 2750 4350
+Wire Wire Line
+	1750 4350 2250 4350
+Wire Wire Line
+	2250 4150 1750 4150
+$Comp
+L Device:C_Small C?
+U 1 1 669A1698
+P 1750 4250
+F 0 "C?" H 1842 4296 50  0000 L CNN
+F 1 "0.1uF" H 1842 4205 50  0000 L CNN
+F 2 "" H 1750 4250 50  0001 C CNN
+F 3 "~" H 1750 4250 50  0001 C CNN
+	1    1750 4250
+	1    0    0    -1
+$EndComp
+Wire Wire Line
+	2750 4350 2500 4350
+Wire Wire Line
+	2500 4150 2750 4150
+Wire Wire Line
+	3250 4350 2750 4350
+Wire Wire Line
+	2750 4150 3250 4150
+$Comp
+L Device:C_Small C?
 U 1 1 66996DA4
 P 3250 4250
 F 0 "C?" H 3342 4296 50  0000 L CNN
-F 1 "C_Small" H 3342 4205 50  0000 L CNN
+F 1 "10uF" H 3342 4205 50  0000 L CNN
 F 2 "" H 3250 4250 50  0001 C CNN
 F 3 "~" H 3250 4250 50  0001 C CNN
@@
 $EndComp
 $Comp
-L Device:C_Small C?
-U 1 1 66998AAD
-P 2750 4250
-F 0 "C?" H 2842 4296 50  0000 L CNN
-F 1 "C_Small" H 2842 4205 50  0000 L CNN
-F 2 "" H 2750 4250 50  0001 C CNN
-F 3 "~" H 2750 4250 50  0001 C CNN
-	1    2750 4250
-	1    0    0    -1
-$EndComp
-$Comp
-L Device:C_Small C?
-U 1 1 669A1692
-P 2250 4250
-F 0 "C?" H 2342 4296 50  0000 L CNN
-F 1 "C_Small" H 2342 4205 50  0000 L CNN
-F 2 "" H 2250 4250 50  0001 C CNN
-F 3 "~" H 2250 4250 50  0001 C CNN
-	1    2250 4250
-	1    0    0    -1
-$EndComp
-$Comp
-L Device:C_Small C?
-U 1 1 669A1698
-P 1750 4250
-F 0 "C?" H 1842 4296 50  0000 L CNN
-F 1 "C_Small" H 1842 4205 50  0000 L CNN
-F 2 "" H 1750 4250 50  0001 C CNN
-F 3 "~" H 1750 4250 50  0001 C CNN
-	1    1750 4250
-	1    0    0    -1
-$EndComp
-Wire Wire Line
-	2500 4150 2250 4150
-Connection ~ 2250 4150
-Wire Wire Line
-	2250 4150 1750 4150
+L power:+5V #PWR?
+U 1 1 669A5A13
+P 3550 2750
+F 0 "#PWR?" H 3550 2600 50  0001 C CNN
+F 1 "+5V" H 3565 2923 50  0000 C CNN
+F 2 "" H 3550 2750 50  0001 C CNN
+F 3 "" H 3550 2750 50  0001 C CNN
+	1    3550 2750
+	1    0    0    -1
+$EndComp
+Wire Wire Line
+	3800 2750 3550 2750
+$Comp
+L Device:Crystal_GND24_Small Y?
+U 1 1 669A8401
+P 3300 2250
+F 0 "Y?" V 3254 2394 50  0000 L CNN
+F 1 "16MHz" V 3345 2394 50  0000 L CNN
+F 2 "" H 3300 2250 50  0001 C CNN
+F 3 "~" H 3300 2250 50  0001 C CNN
+	1    3300 2250
+	0    1    1    0
+$EndComp
+Wire Wire Line
+	3800 2350 3300 2350
+Wire Wire Line
+	3800 2150 3300 2150
+$Comp
+L Device:C_Small C?
+U 1 1 669AB952
+P 2900 2000
+F 0 "C?" V 2671 2000 50  0000 C CNN
+F 1 "22pF" V 2762 2000 50  0000 C CNN
+F 2 "" H 2900 2000 50  0001 C CNN
+F 3 "~" H 2900 2000 50  0001 C CNN
+	1    2900 2000
+	0    1    1    0
+$EndComp
+$Comp
+L Device:C_Small C?
+U 1 1 669ACCC9
+P 2900 2450
+F 0 "C?" V 2671 2450 50  0000 C CNN
+F 1 "22pF" V 2762 2450 50  0000 C CNN
+F 2 "" H 2900 2450 50  0001 C CNN
+F 3 "~" H 2900 2450 50  0001 C CNN
+	1    2900 2450
+	0    1    1    0
+$EndComp
+$Comp
+L power:GND #PWR?
+U 1 1 669ADD8F
+P 2700 2550
+F 0 "#PWR?" H 2700 2300 50  0001 C CNN
+F 1 "GND" H 2705 2377 50  0000 C CNN
+F 2 "" H 2700 2550 50  0001 C CNN
+F 3 "" H 2700 2550 50  0001 C CNN
+	1    2700 2550
+	1    0    0    -1
+$EndComp
+Wire Wire Line
+	3300 2350 3000 2350
+Wire Wire Line
+	3000 2350 3000 2450
+Connection ~ 3300 2350
+Wire Wire Line
+	2800 2000 2700 2000
+Wire Wire Line
+	2700 2000 2700 2450
+Wire Wire Line
+	2800 2450 2700 2450
+Connection ~ 2700 2450
+Wire Wire Line
+	2700 2450 2700 2550
+Wire Wire Line
+	3000 2000 3000 2150
+Wire Wire Line
+	3000 2150 3300 2150
+Connection ~ 3300 2150
+Wire Wire Line
+	3200 2250 3100 2250
+Wire Wire Line
+	3100 2250 3100 2450
+Wire Wire Line
+	3100 2550 2700 2550
+Connection ~ 2700 2550
+Wire Wire Line
+	3400 2250 3400 2450
+Wire Wire Line
+	3400 2450 3100 2450
+Connection ~ 3100 2450
+Wire Wire Line
+	3100 2450 3100 2550
+$Comp
+L Switch:SW_Push SW?
+U 1 1 669B3EA7
+P 3500 1950
+F 0 "SW?" H 3500 2235 50  0000 C CNN
+F 1 "SW_Push" H 3500 2144 50  0000 C CNN
+F 2 "" H 3500 2150 50  0001 C CNN
+F 3 "~" H 3500 2150 50  0001 C CNN
+	1    3500 1950
+	1    0    0    -1
+$EndComp
+$Comp
+L power:GND #PWR?
+U 1 1 669B4CE4
+P 3150 1900
+F 0 "#PWR?" H 3150 1650 50  0001 C CNN
+F 1 "GND" H 3155 1727 50  0000 C CNN
+F 2 "" H 3150 1900 50  0001 C CNN
+F 3 "" H 3150 1900 50  0001 C CNN
+	1    3150 1900
+	1    0    0    -1
+$EndComp
+Wire Wire Line
+	3800 1950 3750 1950
+Wire Wire Line
+	3300 1950 3250 1950
+Wire Wire Line
+	3250 1950 3250 1900
+Wire Wire Line
+	3250 1900 3150 1900
+$Comp
+L power:+5V #PWR?
+U 1 1 669B8397
+P 3750 1500
+F 0 "#PWR?" H 3750 1350 50  0001 C CNN
+F 1 "+5V" H 3765 1673 50  0000 C CNN
+F 2 "" H 3750 1500 50  0001 C CNN
+F 3 "" H 3750 1500 50  0001 C CNN
+	1    3750 1500
+	1    0    0    -1
+$EndComp
+Wire Wire Line
+	3750 1500 3750 1600
+Wire Wire Line
+	3750 1800 3750 1950
+Connection ~ 3750 1950
+Wire Wire Line
+	3750 1950 3700 1950
+$Comp
+L Device:R_Small R?
+U 1 1 669B75BB
+P 3750 1700
+F 0 "R?" H 3809 1746 50  0000 L CNN
+F 1 "10k" H 3809 1655 50  0000 L CNN
+F 2 "" H 3750 1700 50  0001 C CNN
+F 3 "~" H 3750 1700 50  0001 C CNN
+	1    3750 1700
+	1    0    0    -1
+$EndComp
+Text GLabel 2500 2950 0    50   Input ~ 0
+D+
+Text GLabel 2500 3050 0    50   Input ~ 0
+D-
 $EndSCHEMATC
