File: ai03-pcb-guide.kicad_pcb (KiCad board)
At the start: 2 copper layers, 85.7 x 38.1 mm, 24 parts, among them SW1 SW_Push, U1 ATmega32U4-AU, Y1 16MHz

Commit message: PCB Progress
Parts:
- C1, C2, C3, C4, C5, C6, C7, D1, D2, D3, D4, F1, R1, R2, R3, R4, SW1, U1, USB1, Y1: moved to B.Cu
- moved C2 10.6 mm to (79.5, 29.5)
- moved C1 9.82 mm to (88.9, 30.0)
- moved C3 4.13 mm to (70.6, 42.8)
- moved R3 3.86 mm to (59.7, 35.1)
- moved SW1 3.30 mm to (60.7, 51.8), turned to 180 degrees
- moved Y1 2.61 mm to (83.9, 29.9), turned to 180 degrees
- moved C4 2.55 mm to (76.7, 33.3)
- moved R1 2.43 mm to (72.5, 33.2), turned to 90 degrees
- moved R2 2.25 mm to (62.5, 35.1)
- turned R4 to 90 degrees
Connections:
- F1 pad 1: Net-(F1-Pad1) -> +5V
Routing:
- net +5V: track 0.00 -> 102.7 mm, vias 0 -> 6
- net GND: track 0.00 -> 102.0 mm, vias 0 -> 2
- net Net-(R1-Pad2): track 0.00 -> 35.1 mm, vias 0 -> 2
- net Net-(C2-Pad1): track 0.00 -> 14.5 mm
- net VCC: track 0.00 -> 12.9 mm
- net Net-(C1-Pad1): track 0.00 -> 12.6 mm
- net Net-(C3-Pad1): track 0.00 -> 6.83 mm
- net Net-(R3-Pad1): track 20.8 -> 25.8 mm
- net Net-(R4-Pad2): track 0.00 -> 3.96 mm
- net Net-(R2-Pad1): track 21.6 -> 25.0 mm
- net D+: track 5.49 -> 4.70 mm
- net D-: track 5.40 -> 4.69 mm

Commit message: Finalized PCB Design
Parts:
- moved C7 8.83 mm to (71.1, 50.0), turned to 270 degrees
- moved R1 1.52 mm to (73.9, 32.6), turned to 270 degrees
- moved USB1 0.13 mm to (61.4, 25.5)
Connections:
- U1 pad 27: Net-(U1-Pad27) -> ROW0
- U1 pad 28: Net-(U1-Pad28) -> COL1
- U1 pad 29: Net-(U1-Pad29) -> COL0
- U1 pad 30: Net-(U1-Pad30) -> ROW1
- USB1 pad 6: Net-(USB1-Pad6) -> GND
Routing:
- net GND: track 102.0 -> 167.2 mm, vias 2 -> 0
- net ROW1: track 0.00 -> 52.8 mm
- net COL1: track 0.00 -> 52.3 mm
- net ROW0: track 0.00 -> 48.0 mm
- net COL0: track 0.00 -> 33.1 mm
- net +5V: track 102.7 -> 111.0 mm
- net Net-(D3-Pad2): track 0.00 -> 7.23 mm
- net Net-(D1-Pad2): track 0.00 -> 7.23 mm
- net Net-(D4-Pad2): track 0.00 -> 7.23 mm
- net Net-(D2-Pad2): track 0.00 -> 7.23 mm
- net Net-(R1-Pad2): track 35.1 -> 36.0 mm
- added copper zone on B.Cu, net GND
Other:
- board text added: "TyKeys"
